File: scart adapter/rgb2scart.sch (EAGLE design)
At the start: 10 parts, among them J1 AUDIO_JACK_3.5MM_PTH, X1 SCART-F

Commit message: Add files via upload
Parts:
- removed P_BLUE, P_GREEN, P_RED: (no value), pot:TRIM_US-PT-10
- added C1, C2: 0.1uF, SparkFun-Capacitors:0.1UF-KIT-EZ-50V-20%
- added IC1: LM1881N, oldchips2:LM1881N
- added IC3: REG1117, burr-brown-5:REG1117
- added JP1: (no value), jumper:JP2E
- added R3, R4, R5: (no value), bourns:3362P
- added R6: 390, SparkFun-Resistors:1KOHM-HORIZ-1/4W-1%
Connections:
- new net 5V: IC1P.VCC, IC3.VOUT
- new net CSYNC: IC1G$1.CSYNC, JP1.1
- new net N$1: JP1.2, R1.2
- new net N$4: C2.1, IC1G$1.RSET, R6.1
- new net N$5: C1.2, IC1G$1.VIDEO
- new net VSYNC: IC1G$1.VS
- net 12V: now also IC3.VIN
- net GND: now also C2.2, IC1P.GND, IC3.GND, R3.1, R4.1, R5.1, R6.2; no longer P_BLUE.A, P_GREEN.A, P_RED.A
- net IN_BLUE: now also R5.3; no longer P_BLUE.E
- net IN_GREEN: now also C1.1, R4.3; no longer P_GREEN.E
- net IN_RED: now also R3.3; no longer P_RED.E
- net OUT_BLUE: now also R5.2; no longer P_BLUE.S
- net OUT_GREEN: now also R4.2; no longer P_GREEN.S
- net OUT_RED: now also R3.2; no longer P_RED.S
- net SYNC: now also JP1.3; no longer R1.2
